File: WELLER.kicad_pcb (KiCad board)
At the start: 2 copper layers, 20 x 100 mm, 55 parts, among them J1 Jack-DC, J2 AudioJack3_Ground_SwitchTR, J3 jtag conector, Q1 DMP2018LFK, SW1 SW_Push_SPDT, SW2 SW_Push, SW3 SW_Push, U1 AP1117-33, U2 LTC4440ES6, U3 MCP603-xCH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

Commit message: duży update, gotowe pcb
Parts:
- removed R16: 10R, Resistor_SMD:R_0603_1608Metric
- removed U5: STM32F031K6Ux, Package_DFN_QFN:QFN-32-1EP_5x5mm_P0.5mm_EP3.45x3.45mm
- added C11: n.c., Capacitor_SMD:C_0603_1608Metric, F.Cu at (136.3, 54.9)
- added C20: 100n, Capacitor_SMD:C_0603_1608Metric_Pad1.05x0.95mm_HandSolder, F.Cu at (130.5, 66.5)
- added J4: Conn_01x04_Female, Connector_PinHeader_2.54mm:PinHeader_1x04_P2.54mm_Vertical, F.Cu at (125.7, 72.1)
- added R14: n.c., Resistor_SMD:R_0603_1608Metric_Pad1.05x0.95mm_HandSolder, F.Cu at (126.8, 67.9)
- R7: footprint Resistor_SMD:R_0402_1005Metric -> Resistor_SMD:R_0603_1608Metric
- moved C13 15.2 mm to (121.9, 60.5), turned to 180 degrees
- moved C9 14.6 mm to (131.9, 51.6), turned to 90 degrees
- moved H3 14.0 mm to (125.1, 92.4)
- moved C6 13.6 mm to (137.9, 38.5), turned to 180 degrees
- moved C16 13.1 mm to (129.4, 51.7), turned to 135 degrees
- moved C14 12.1 mm to (128.3, 52.8), turned to 135 degrees
- moved C17 11.6 mm to (136.0, 63.3), turned to 135 degrees
- moved R4 10.2 mm to (128.2, 88.2)
- moved D5 10.0 mm to (131.8, 88.1), turned to 180 degrees
- moved J3 9.85 mm to (126.6, 65.3), turned to 180 degrees
- moved R12 9.07 mm to (138.6, 55.7), turned to 90 degrees
- moved R5 7.95 mm to (121.0, 75.2), turned to 270 degrees
- moved R2 7.65 mm to (128.3, 83.5)
- moved D3 7.52 mm to (131.8, 83.5), turned to 180 degrees
- moved C10 6.80 mm to (133.7, 51.6), turned to 90 degrees
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Connections:
- C10 pad 1: GNDA -> GND
- C17 pad 1: GNDA -> GND
- C17 pad 2: /stm32/3_3v_analog -> /tip_driving/3.3V_analog
- C9 pad 1: GNDA -> GND
- J3 pad 1: /tip_driving/3.3V_analog -> (no net)
- J3 pad 6: Net-(J3-Pad6) -> (no net)
- J3 pad 8: Net-(J3-Pad8) -> (no net)
- U3 pad 2: GNDA -> GND
- U4 pad 11: Net-(U4-Pad11) -> (no net)
- U4 pad 12: Net-(U4-Pad12) -> (no net)
- U4 pad 13: Net-(U4-Pad13) -> (no net)
- U4 pad 14: Net-(U4-Pad14) -> (no net)
- U4 pad 15: Net-(U4-Pad15) -> (no net)
- U4 pad 16: Net-(U4-Pad16) -> (no net)
- U4 pad 17: Net-(U4-Pad17) -> (no net)
- U4 pad 18: /stm32/led_g -> (no net)
- U4 pad 19: /stm32/led_r -> (no net)
- U4 pad 20: /stm32/led_y -> (no net)
- U4 pad 21: Net-(U4-Pad21) -> (no net)
- U4 pad 22: Net-(U4-Pad22) -> (no net)
- U4 pad 25: Net-(U4-Pad25) -> (no net)
- U4 pad 26: Net-(U4-Pad26) -> (no net)
- U4 pad 27: Net-(U4-Pad27) -> (no net)
- U4 pad 28: Net-(U4-Pad28) -> (no net)
- U4 pad 30: Net-(U4-Pad30) -> (no net)
- U4 pad 31: Net-(U4-Pad31) -> (no net)
- U4 pad 32: Net-(U4-Pad32) -> (no net)
- U4 pad 33: Net-(U4-Pad33) -> (no net)
- U4 pad 38: Net-(U4-Pad38) -> (no net)
- U4 pad 39: Net-(U4-Pad39) -> /stm32/led_g
- U4 pad 4: Net-(U4-Pad4) -> (no net)
- U4 pad 40: Net-(U4-Pad40) -> /stm32/led_r
- U4 pad 41: Net-(U4-Pad41) -> /stm32/led_y
- U4 pad 42: Net-(U4-Pad42) -> /stm32/scl
- U4 pad 43: Net-(U4-Pad43) -> /stm32/sda
- U4 pad 45: Net-(U4-Pad45) -> (no net)
- U4 pad 46: Net-(U4-Pad46) -> (no net)
- U4 pad 6: Net-(U4-Pad6) -> (no net)
- U4 pad 8: GNDA -> GND
- U4 pad 9: /stm32/3_3v_analog -> /tip_driving/3.3V_analog
Routing:
- net /tip_driving/12V: track 0.00 -> 132.7 mm, vias 0 -> 7
- net /tip_driving/3.3V_analog: track 0.00 -> 110.3 mm, vias 27 -> 32
- net /tip_driving/heater: track 0.00 -> 38.4 mm, vias 1 -> 14
- net /stm32/led_g: track 0.00 -> 29.2 mm
- net /but_led/sw1: track 0.00 -> 28.5 mm, vias 0 -> 2
- net GND: track 0.00 -> 25.9 mm, vias 0 -> 122
- net /stm32/weller_con1: track 0.00 -> 24.4 mm, vias 0 -> 2
- net /stm32/led_r: track 0.00 -> 24.0 mm
- net /stm32/sda: track 0.00 -> 19.3 mm
- net /stm32/led_y: track 0.00 -> 19.2 mm
- net Net-(C6-Pad1): track 0.00 -> 14.8 mm
- net /but_led/sw2: track 0.00 -> 12.5 mm
- net Net-(R10-Pad2): track 0.00 -> 12.3 mm
- net /stm32/scl: track 0.00 -> 11.8 mm
- net /stm32/SWDIO: track 0.00 -> 10.9 mm, vias 0 -> 1
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- added copper zone on B.Cu, net GND
- added copper zone on F.Cu, net GND
