File: mcu.sch (KiCad schematic (older format))
At the start: 17 parts, among them J3 debug+programing, J4 I2c oled, U4 STM32F103C8Tx, U5 SM353LT

Commit message: update front endu do termopary i przełącznika zasilającego
Other:
- note added: "OLED 0,91' 4P 128x32 na I2C - SSD1306"
- note added: "TEMP_SENSOR ?"
- note added: "Wyprowadzenie pinów na test pointy ?"
- moved on the sheet: R16
Changed lines of the file:
@@
 Wire Wire Line
 	6600 1200 6700 1200
-Text HLabel 4500 1850 1    50   Input ~ 0
+Text HLabel 4500 1850 1    50   Input ~ 6
 3_3_stm
-Text Label 6900 1600 0    50   ~ 0
+Text Label 6900 1600 0    50   ~ 6
 3_3v_analog
 $Comp
@@
 Wire Wire Line
 	4600 3050 4600 2950
-Text HLabel 6700 1050 1    50   Input ~ 0
+Text HLabel 6700 1050 1    50   Input ~ 6
 3_3_stm
 Wire Wire Line
@@
 Wire Wire Line
 	4350 1850 4350 2000
-Text HLabel 5850 3100 0    50   BiDi ~ 0
+Text HLabel 5850 3100 0    50   BiDi ~ 6
 sw1
-Text HLabel 5850 3200 0    50   BiDi ~ 0
+Text HLabel 5850 3200 0    50   BiDi ~ 6
 sw2
-Text HLabel 5750 3800 0    50   Output ~ 0
+Text HLabel 5750 3800 0    50   Output ~ 6
 led_g
-Text HLabel 5750 3900 0    50   Output ~ 0
+Text HLabel 5750 3900 0    50   Output ~ 6
 led_r
-Text HLabel 5750 4000 0    50   Output ~ 0
+Text HLabel 5750 4000 0    50   Output ~ 6
 led_y
-Text HLabel 5650 3600 0    50   BiDi ~ 0
+Text HLabel 5650 3600 0    50   BiDi ~ 6
 weller_con1
-Text HLabel 7650 4600 2    50   Output ~ 0
+Text HLabel 7650 4600 2    50   Output ~ 6
 PWM_heater
 Wire Wire Line
@@
 Wire Wire Line
 	7300 4900 7650 4900
-Text Label 7650 4800 0    50   ~ 0
+Text Label 7650 4800 0    50   ~ 6
 SWDIO
-Text Label 7650 4900 0    50   ~ 0
+Text Label 7650 4900 0    50   ~ 6
 SWCLK
-Text Label 5750 2400 0    50   ~ 0
+Text Label 5750 2400 0    50   ~ 6
 nRST
 Wire Wire Line
@@
 Wire Wire Line
 	6500 5500 6600 5500
-Text Label 1900 6850 0    50   ~ 0
+Text Label 1900 6850 0    50   ~ 6
 nRST
-Text Label 1900 6450 0    50   ~ 0
+Text Label 1900 6450 0    50   ~ 6
 SWDIO
-Text Label 1900 6550 0    50   ~ 0
+Text Label 1900 6550 0    50   ~ 6
 SWCLK
 Connection ~ 6900 1950
@@
 Wire Wire Line
 	6700 1650 6700 2200
-Text Label 5650 2600 0    50   ~ 0
+Text Label 5650 2600 0    50   ~ 6
 BOOT
 $Comp
@@
 L power:GND #PWR0139
 U 1 1 5CEC799A
-P 1450 3900
-F 0 "#PWR0139" H 1450 3650 50  0001 C CNN
-F 1 "GND" H 1455 3727 50  0000 C CNN
-F 2 "" H 1450 3900 50  0001 C CNN
-F 3 "" H 1450 3900 50  0001 C CNN
-	1    1450 3900
-	1    0    0    -1
-$EndComp
-Wire Wire Line
-	1550 3900 1450 3900
-Text HLabel 1400 3800 0    50   Input ~ 0
+P 1100 3900
+F 0 "#PWR0139" H 1100 3650 50  0001 C CNN
+F 1 "GND" H 1105 3727 50  0000 C CNN
+F 2 "" H 1100 3900 50  0001 C CNN
+F 3 "" H 1100 3900 50  0001 C CNN
+	1    1100 3900
+	1    0    0    -1
+$EndComp
+Wire Wire Line
+	1550 3900 1100 3900
+Text HLabel 1100 3800 0    50   Input ~ 6
 3_3_stm
 Wire Wire Line
-	1400 3800 1550 3800
-Wire Wire Line
-	1550 3700 1450 3700
-Wire Wire Line
-	1550 3600 1400 3600
-Text Label 1400 3600 0    50   ~ 0
+	1100 3800 1550 3800
+Wire Wire Line
+	1550 3700 1300 3700
+Wire Wire Line
+	1550 3600 1100 3600
+Text Label 1100 3600 0    50   ~ 6
 sda
-Text Label 1400 3700 0    50   ~ 0
+Text Label 1100 3700 0    50   ~ 6
 scl
-Text Label 5750 4200 0    50   ~ 0
+Text Label 5750 4200 0    50   ~ 6
 sda
 Wire Wire Line
 	5750 4200 6000 4200
-Text Label 5750 4100 0    50   ~ 0
+Text Label 5750 4100 0    50   ~ 6
 scl
 Wire Wire Line
@@
 L Device:R R16
 U 1 1 5CEC6FCF
-P 1450 3550
-F 0 "R16" H 1520 3596 50  0000 L CNN
-F 1 "10k" H 1520 3505 50  0000 L CNN
-F 2 "Resistor_SMD:R_0603_1608Metric" V 1380 3550 50  0001 C CNN
-F 3 "~" H 1450 3550 50  0001 C CNN
-	1    1450 3550
-	1    0    0    -1
-$EndComp
-Connection ~ 1450 3700
-Wire Wire Line
-	1450 3700 1400 3700
-Text HLabel 1400 3300 0    50   Input ~ 0
+P 1300 3550
+F 0 "R16" H 1370 3596 50  0000 L CNN
+F 1 "10k" H 1370 3505 50  0000 L CNN
+F 2 "Resistor_SMD:R_0603_1608Metric" V 1230 3550 50  0001 C CNN
+F 3 "~" H 1300 3550 50  0001 C CNN
+	1    1300 3550
+	1    0    0    -1
+$EndComp
+Connection ~ 1300 3700
+Wire Wire Line
+	1300 3700 1100 3700
+Text HLabel 1150 3300 0    50   Input ~ 6
 3_3_stm
 Wire Wire Line
-	1400 3300 1450 3300
-Wire Wire Line
-	1450 3300 1450 3400
-Wire Wire Line
-	1450 3300 1550 3300
-Connection ~ 1450 3300
+	1150 3300 1300 3300
+Wire Wire Line
+	1300 3300 1300 3400
+Wire Wire Line
+	1300 3300 1550 3300
+Connection ~ 1300 3300
 $Comp
 L Connector_Generic:Conn_02x05_Odd_Even J3
@@
 Wire Wire Line
 	7400 3800 7300 3800
-Text HLabel 7400 3800 2    50   Input ~ 0
+Text HLabel 7400 3800 2    50   Input ~ 6
 termocouple
 NoConn ~ 7300 3700
@@
 	-1   0    0    -1
 $EndComp
-Text Label 7650 3500 2    50   ~ 0
+Text Label 7650 3500 2    50   ~ 6
 hall_in
 Wire Wire Line
 	7300 3500 7650 3500
-Text Label 1150 5200 2    50   ~ 0
+Text Label 1150 5200 2    50   ~ 6
 hall_in
 $Comp
@@
 Wire Wire Line
 	1800 4900 1800 4850
-Text HLabel 1800 4800 1    50   Input ~ 0
+Text HLabel 1800 4800 1    50   Input ~ 6
 3_3_stm
 Wire Wire Line
 	1150 5200 1200 5200
-Text HLabel 1200 6450 0    50   Input ~ 0
+Text HLabel 1200 6450 0    50   Input ~ 6
 3_3_stm
 $Comp
@@
 Wire Wire Line
 	7300 4300 7650 4300
-Text Label 7650 4300 2    50   ~ 0
+Text Label 7650 4300 2    50   ~ 6
 usart_rx
-Text Label 7650 4400 2    50   ~ 0
+Text Label 7650 4400 2    50   ~ 6
 usart_tx
-Text Label 7650 4500 2    50   ~ 0
+Text Label 7650 4500 2    50   ~ 6
 usart_ck
 Wire Wire Line
@@
 Wire Wire Line
 	7300 4400 7650 4400
-Text Label 1200 6550 2    50   ~ 0
+Text Label 1200 6550 2    50   ~ 6
 usart_rx
-Text Label 1200 6650 2    50   ~ 0
+Text Label 1200 6650 2    50   ~ 6
 usart_tx
-Text Label 1200 6750 2    50   ~ 0
+Text Label 1200 6750 2    50   ~ 6
 usart_ck
 Wire Wire Line
@@
 Wire Wire Line
 	7400 3600 7300 3600
-Text HLabel 7400 3600 2    50   Input ~ 0
+Text HLabel 7400 3600 2    50   Input ~ 6
 input_sense
 NoConn ~ 7300 3900
@@
 	1    0    0    -1
 $EndComp
+Text Notes 750  3150 0    50   ~ 6
+OLED 0,91' 4P 128x32 na I2C - SSD1306
+Text Notes 1250 2050 0    50   ~ 6
+TEMP_SENSOR ?
+Text Notes 8400 3250 0    50   ~ 6
+Wyprowadzenie pinów na test pointy ?
+Wire Notes Line
+	8500 3300 8500 3950
+Wire Notes Line
+	8500 3950 8050 3950
 $EndSCHEMATC
